Commit message: easter updates

File: descriptions/robot_descriptions/objects_description/objects/table.urdf (robot description, URDF)
Before this commit: robot table, 7 links, 6 joints
Links:
- link table_top_link: geometry collision box size=2.0 3.0 0.05; visual box size=2.0 3.0 0.05

Commit message: new data plus new GMM and different optimisation - Harshit

File: descriptions/robot_descriptions/objects_description/objects/table.urdf (robot description, URDF)
Before this commit: robot table, 7 links, 6 joints
Links:
- link table_top_link: geometry collision box size=2.0 1.8 0.05; visual box size=2.0 1.8 0.05
Joints:
- joint table_leg1_joint: origin xyz=0.455 0.70 -0.05 rpy=0 0 0 -> xyz=0.91 0.80 -0.05 rpy=0 0 0
- joint table_leg2_joint: origin xyz=0.455 -0.70 -0.05 rpy=0 0 0 -> xyz=0.91 -0.80 -0.05 rpy=0 0 0
- joint table_leg3_joint: origin xyz=-0.455 -0.70 -0.05 rpy=0 0 0 -> xyz=-0.91 -0.80 -0.05 rpy=0 0 0
- joint table_leg4_joint: origin xyz=-0.455 0.70 -0.05 rpy=0 0 0 -> xyz=-0.91 0.80 -0.05 rpy=0 0 0
