Commit message: 10 dof robot

File: descriptions/robot_descriptions/objects_description/objects/robot10.urdf (robot description, URDF)
Before this commit: robot robot_arm_10_joints, 11 links, 10 joints
Links:
- link link_1: mass None -> 5.0; geometry collision cylinder length=0.1 radius=0.05; visual cylinder length=0.1 radius=0.05
- link link_10: mass None -> 2.3466; geometry collision cylinder length=0.1 radius=0.05; visual cylinder length=0.1 radius=0.05
- link link_2: mass None -> 3.4525; geometry collision cylinder length=0.1 radius=0.05; visual cylinder length=0.1 radius=0.05
- link link_3: mass None -> 3.4821; geometry collision cylinder length=0.1 radius=0.05; visual cylinder length=0.1 radius=0.05
- link link_4: mass None -> 4.05623; geometry collision cylinder length=0.1 radius=0.05; visual cylinder length=0.1 radius=0.05
- link link_5: mass None -> 3.4822; geometry collision cylinder length=0.1 radius=0.05; visual cylinder length=0.1 radius=0.05
- link link_6: mass None -> 2.1633; geometry collision cylinder length=0.1 radius=0.05; visual cylinder length=0.1 radius=0.05
- link link_7: mass None -> 2.3466; geometry collision cylinder length=0.1 radius=0.05; visual cylinder length=0.1 radius=0.05
- link link_8: mass None -> 2.3466; geometry collision cylinder length=0.1 radius=0.05; visual cylinder length=0.1 radius=0.05
- link link_9: mass None -> 2.3466; geometry collision cylinder length=0.1 radius=0.05; visual cylinder length=0.1 radius=0.05

Commit message: 10 dof robot

File: descriptions/robot_descriptions/objects_description/objects/robot10.urdf (robot description, URDF)
Before this commit: robot robot_arm_10_joints, 11 links, 10 joints
Joints:
- joint joint_10: axis 0 0 1 -> 1 0 0

Commit message: .

File: descriptions/robot_descriptions/objects_description/objects/robot10.urdf (robot description, URDF)
Before this commit: robot robot_arm_10_joints, 11 links, 10 joints
Joints:
- joint joint_7: axis 0 0 1 -> 0 1 0
- joint joint_8: axis 0 1 0 -> 1 0 0
